Commit message: fix geometry

File: tm_description/xacro/macro.tm12-nominal.urdf.xacro (robot description, xacro)
@@ -232,6 +232,9 @@
     <collision>
       <geometry>
+        <mesh filename="package://tm_description/meshes/tm5-900/visual/tmr_100w_01.stl" />
+      </geometry>
+      <!-- <geometry>
         <mesh filename="package://tm_description/meshes/tm5-900/collision/tmr_100w_01_c.stl" />
-      </geometry>
+      </geometry> -->
     </collision>
     <inertial>
@@ -302,6 +305,9 @@
     <collision>
       <geometry>
+        <mesh filename="package://tm_description/meshes/tm5-900/visual/tmr_ee.stl" />
+      </geometry>
+      <!-- <geometry>
         <mesh filename="package://tm_description/meshes/tm5-900/collision/tmr_ee_c.stl" />
-      </geometry>
+      </geometry> -->
     </collision>
     <inertial>
